Commit message: fix json to csv for pi tripedal code

File: 3_simulation/tripedal_robot.urdf (robot description, URDF)
Before this commit: robot tripedal_robot, 10 links, 9 joints
Links:
- link center_foot: mass 0.1 -> 0.5
- link center_leg_part1: mass 0.1 -> 0.3
- link center_leg_part2: mass 0.1 -> 0.5
- link left_foot: mass 0.1 -> 0.3
- link left_leg_lower: mass 0.1 -> 0.3
- link left_leg_upper: mass 0.1 -> 0.3
- link right_foot: mass 0.1 -> 0.3
- link right_leg_lower: mass 0.1 -> 0.3
- link right_leg_upper: mass 0.1 -> 0.3
