Commit message: trained model

File: 3_simulation/better_tripedal_robot.urdf (robot description, URDF)
Before this commit: robot better_tripedal_robot, 10 links, 9 joints
Links:
- link center_foot: geometry collision cylinder length=0.02 radius=0.13; visual cylinder length=0.02 radius=0.13
- link left_foot: mass 0.3 -> 0.5; geometry collision box size=0.12 0.18 0.05; visual box size=0.12 0.18 0.05
- link right_foot: mass 0.3 -> 0.5; geometry collision box size=0.12 0.18 0.05; visual box size=0.12 0.18 0.05
Joints:
- joint center_foot_joint: origin xyz=0 0 -0.2 rpy=0 0 0 -> xyz=0 0 -0.24 rpy=0 0 0
- joint left_foot_joint: origin xyz=0 0 -0.23 rpy=0 0 0 -> xyz=0 0 -0.25 rpy=0 0 0
- joint left_hip: limit lower=-1.57 upper=1.57 effort=10 velocity=10 -> lower=-2.617 upper=2.617 effort=10 velocity=10
- joint left_knee: limit lower=-2 upper=2 effort=10 velocity=10 -> lower=-2.356 upper=2.356 effort=10 velocity=10
- joint right_foot_joint: origin xyz=0 0 -0.23 rpy=0 0 0 -> xyz=0 0 -0.25 rpy=0 0 0
- joint right_hip: limit lower=-1.57 upper=1.57 effort=10 velocity=10 -> lower=-2.617 upper=2.617 effort=10 velocity=10
- joint right_knee: limit lower=-2 upper=2 effort=10 velocity=10 -> lower=-2.356 upper=2.356 effort=10 velocity=10
